File: ESP-32/ESP-32.kicad_sch (KiCad schematic)
At the start: 20 parts, among them J1 USB_B_Micro, J2 Conn_01x21_Pin, J3 Conn_01x21_Pin, U2 esp32-devkitM-1

Commit message: DSD
Parts:
- added C10, C11, C9: 0.1uF, Capacitor_SMD:C_0805_2012Metric_Pad1.18x1.45mm_HandSolder, symbol Device:C
- added C7, C8: 10uF, Capacitor_SMD:C_0805_2012Metric_Pad1.18x1.45mm_HandSolder, symbol Device:C
- added D5: LED, LED_SMD:LED_0805_2012Metric_Pad1.15x1.40mm_HandSolder, symbol Device:LED
- added Q1, Q2: 2SC4213, Package_TO_SOT_SMD:SOT-323_SC-70, symbol Transistor_BJT:2SC4213
- added R11: 5.1K, Resistor_SMD:R_0805_2012Metric_Pad1.20x1.40mm_HandSolder, symbol Device:R
- added R7: 47.5K, Resistor_SMD:R_0805_2012Metric_Pad1.20x1.40mm_HandSolder, symbol Device:R
- added R8, R9: 10K, Resistor_SMD:R_0805_2012Metric_Pad1.20x1.40mm_HandSolder, symbol Device:R
- added SW1, SW2: SW_Omron_B3FS, Button_Switch_SMD:SW_SPST_PTS810, symbol Switch:SW_Omron_B3FS
- added U1: CP2102N-Axx-xQFN28, Package_DFN_QFN:QFN-28-1EP_5x5mm_P0.5mm_EP3.35x3.35mm, symbol Interface_USB:CP2102N-Axx-xQFN28
- added U3: LM1117MP-3.3, Package_TO_SOT_SMD:SOT-223-3_TabPin2, symbol Regulator_Linear:LM1117MP-3.3
- C1: value 10uF -> 1uF; footprint (none) -> Capacitor_SMD:C_0805_2012Metric_Pad1.18x1.45mm_HandSolder
- C2: value 22pF -> 10uF; footprint (none) -> Capacitor_SMD:C_0805_2012Metric_Pad1.18x1.45mm_HandSolder
- C3: value 22pF -> 0.1uF; footprint (none) -> Capacitor_SMD:C_0805_2012Metric_Pad1.18x1.45mm_HandSolder
- C4, C5, C6: footprint (none) -> Capacitor_SMD:C_0805_2012Metric_Pad1.18x1.45mm_HandSolder
- D2, D3, D4: footprint TVS_LESD5D5.0CT1G -> LESD5D5.0CT1G:TVS_LESD5D5.0CT1G
- J2, J3: footprint (none) -> Connector_PinSocket_2.54mm:PinSocket_1x17_P2.54mm_Vertical_SMD_Pin1Left; symbol Connector:Conn_01x21_Pin -> Connector:Conn_01x17_Pin
- R1, R2, R5: footprint (none) -> Resistor_SMD:R_0805_2012Metric_Pad1.20x1.40mm_HandSolder
- R3: value 0 -> 10K; footprint (none) -> Resistor_SMD:R_0805_2012Metric_Pad1.20x1.40mm_HandSolder
- R4: value 0 -> 22.1K; footprint (none) -> Resistor_SMD:R_0805_2012Metric_Pad1.20x1.40mm_HandSolder
- R6: value 10K -> 1K; footprint (none) -> Resistor_SMD:R_0805_2012Metric_Pad1.20x1.40mm_HandSolder
- U2: footprint nuevo simbolo:esp32-devkitM-1 -> esp32-devkitM-1:esp32-devkitM-1
Connections:
- net GPIO00 is gone; now on net GPIO0: U2.21 (IO0)
- net GPIO02 is gone; now on net GPIO2: U2.20 (IO2)
- net GPIO04 is gone; now on net GPIO4: U2.22 (IO4)
- net GPIO05 is gone; now on net GPIO5: U2.29 (IO5)
- net GPIO09 is gone; now on net GPIO9: U2.25 (IO9)
- net GPIO11 is gone; now on net GPIO26: J2.13 (Pin_13)
- net GPIO3 is gone; now on net GPIO38: J2.5 (Pin_5)
- net GPIO6 is gone; now on net GPIO34: J2.8 (Pin_8)
- net GPIO7 is gone; now on net GPIO35: J2.9 (Pin_9)
- net GPIO8 is gone; now on net GPIO32: J2.10 (Pin_10)
- net Earth: now also C2.1, C3.1, R3.2, C10.2, C11.1, C7.2, C8.2, C9.2, D5.1 (K), R7.2, SW1.1, SW2.1, U1.29 (GND), U1.3 (GND), U3.1 (GND); no longer C2.2, C3.2
- net GND: now also J2.1 (Pin_1), J2.17 (Pin_17); no longer J2.21 (Pin_21)
- net GPIO0: now also J3.13 (Pin_13), C11.2, Q2.2 (E), SW1.2; no longer J2.2 (Pin_2)
- net GPIO10: now also J3.10 (Pin_10); no longer J2.12 (Pin_12)
- net GPIO12: now also J3.17 (Pin_17); no longer J2.14 (Pin_14)
- net GPIO13: now also J3.16 (Pin_16); no longer J2.15 (Pin_15)
- net GPIO14: now also J2.15 (Pin_15); no longer J2.16 (Pin_16)
- net GPIO15: now also J3.15 (Pin_15); no longer J2.17 (Pin_17)
- net GPIO18: now also J3.8 (Pin_8); no longer R6.2
- net GPIO19: now also J3.6 (Pin_6); no longer C2.1, R3.2
- net GPIO2: now also J3.14 (Pin_14); no longer J2.4 (Pin_4)
- net GPIO21: now also J3.4 (Pin_4)
- net GPIO33: now also J2.11 (Pin_11)
- net GPIO37: now also J2.4 (Pin_4)
- net GPIO39: now also J2.6 (Pin_6)
- net GPIO4: now also J3.12 (Pin_12); no longer J2.6 (Pin_6)
- net GPIO5: now also J3.9 (Pin_9); no longer J2.7 (Pin_7)
- net GPIO9: now also J3.11 (Pin_11); no longer J2.11 (Pin_11)
- net U0RXD: now also J3.2 (Pin_2), R1.2
- net U0TXD: now also J3.3 (Pin_3), R2.2
- net USB_DN: now also D3.2, J1.2 (D-), U1.5 (D-); no longer R4.2
- net USB_DP: now also D4.2, J1.3 (D+), U1.4 (D+); no longer R2.2
- net VBUS: now also D1.2 (A); no longer D1.1 (K)
- net VCC: now also C2.2, D1.1 (K), J2.16 (Pin_16), J2.2 (Pin_2), R4.1, C10.1, C7.1, C8.1, C9.1, R11.1, U1.6 (VDD), U1.7 (VREGIN), U3.2 (VO), U3.3 (VI); no longer C3.1, D1.2 (A), J2.1 (Pin_1), J2.20 (Pin_20)
- net GPIO22: now reaches J3.5 (Pin_5)
- net GPIO22: now also U2.33 (IO22)
- net GPIO23: now reaches J3.7 (Pin_7)
- net GPIO23: now also U2.31 (IO23)
- net GPIO32: now reaches U2.11 (IO32)
- net GPIO25: now reaches U2.13 (IO25)
- net GPIO25: now also J2.12 (Pin_12)
- net GPIO27: now reaches U2.15 (IO27)
- net GPIO27: now also J2.14 (Pin_14)
- net CHIP_PU renamed ESP_RST
- net ESP_RST: now also C3.2, J2.7 (Pin_7), Q1.3 (C), SW2.2
- net GPIO1 renamed GPIO36
- removed net GPIO16: J2.18 (Pin_18)
- removed net GPIO17: J2.19 (Pin_19)
- net GPIO20: no longer names the net of C1.1
- net GPIO20: now also R4.2, R7.1, U1.8 (VBUS); no longer R1.2
- new net: R3.1, U1.11 (~{SUSPEND})
- new net: R2.1, U1.25 (RXD)
- new net: R1.1, U1.26 (TXD)
- new net: R6.2, U1.9 (~{RST})
- new net: Q2.1 (B), R9.2
- new net: Q1.1 (B), R8.2
- new net: D5.2 (A), R11.2
- new net DTR: Q2.3 (C), R8.1, U1.28 (~{DTR})
- new net RTS: Q1.2 (E), R9.1, U1.24 (~{RTS})
- no-connect marks 6 -> 16
Other:
- moved on the sheet: C4, C5, C6, D1, R5

Commit message: pcb actualizado
Parts:
- D1: footprint Diode_THT:D_DO-41_SOD81_P10.16mm_Horizontal -> Diode_SMD:D_0805_2012Metric_Pad1.15x1.40mm_HandSolder
- J2, J3: footprint Connector_PinSocket_2.54mm:PinSocket_1x17_P2.54mm_Vertical_SMD_Pin1Left -> Connector_PinSocket_2.54mm:PinSocket_1x17_P2.54mm_Vertical
Changed lines of the file:
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@@
       (effects (font (size 1.27 1.27)))
     )
-    (property "Footprint" "Connector_PinSocket_2.54mm:PinSocket_1x17_P2.54mm_Vertical_SMD_Pin1Left" (at 297.18 53.34 0)
+    (property "Footprint" "Connector_PinSocket_2.54mm:PinSocket_1x17_P2.54mm_Vertical" (at 297.18 53.34 0)
       (effects (font (size 1.27 1.27)) hide)
     )
@@
       (effects (font (size 1.27 1.27)))
     )
-    (property "Footprint" "Connector_PinSocket_2.54mm:PinSocket_1x17_P2.54mm_Vertical_SMD_Pin1Left" (at 344.17 53.34 0)
+    (property "Footprint" "Connector_PinSocket_2.54mm:PinSocket_1x17_P2.54mm_Vertical" (at 344.17 53.34 0)
       (effects (font (size 1.27 1.27)) hide)
     )
@@
       (effects (font (size 1.27 1.27)))
     )
-    (property "Footprint" "Diode_THT:D_DO-41_SOD81_P10.16mm_Horizontal" (at 44.45 23.495 0)
-      (effects (font (size 1.27 1.27)) hide)
-    )
+    (property "Footprint" "Diode_SMD:D_0805_2012Metric_Pad1.15x1.40mm_HandSolder" (at 44.45 23.495 0)
+      (effects (font (size 1.27 1.27)) hide)
+    )
